File: Projects/Robot Arm/Robot Arm Controller.brd (EAGLE design)
At the start: 160 x 80 mm, 71 parts, among them IC1 U_FTDICHIP_FT232RL, J1 ICSP HEADER, J2 SERVO PWR, J3 STEPPER, J4 J_MOLEX_502386, P1 P_USB_MINIUX60A-MB-5ST, P2 +12V INPUT, Q1 FDV303N, U1 UA78M05CDCY, U2 TPS71550DCKR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

Commit message: Almost done
Parts:
- moved S3 28.4 mm to (28.2, 60.7), turned to 0 degrees
- moved J1 27.2 mm to (7.50, 46.4)
- moved C4 26.8 mm to (25.3, 28.9), turned to 180 degrees
- moved U2 23.9 mm to (21.1, 29.5)
- moved R5 23.2 mm to (40.1, 39.9), turned to 180 degrees
- moved R6 21.1 mm to (37.0, 30.1), turned to 90 degrees
- moved R1 20.4 mm to (22.0, 32.8), turned to 90 degrees
- moved Q1 17.9 mm to (32.7, 46.1)
- moved RN3 16.6 mm to (5.50, 51.1), turned to 270 degrees
- moved C7 15.6 mm to (7.00, 39.4), turned to 90 degrees
- moved C21 15.4 mm to (2.20, 51.0)
- moved S1 15.0 mm to (17.4, 60.7), turned to 180 degrees
- moved C10 14.6 mm to (9.20, 39.4), turned to 90 degrees
- moved R18 12.7 mm to (21.6, 42.3), turned to 180 degrees
- moved C20 12.5 mm to (8.80, 51.1)
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Connections:
- net +5V: now also RN2.3B; no longer RN2.1B
- net N$9: now also RN2.1A; no longer RN2.3A
- net RESET: now also RN2.3A; no longer RN2.1A
- net TX: now also RN2.1B; no longer RN2.3B
Routing:
- net +5V: track 83.9 -> 189.1 mm, vias 1 -> 6
- net N$67: track 0.00 -> 76.0 mm, vias 0 -> 2
- net GND: track 121.4 -> 186.4 mm, vias 16 -> 19
- net HALL_SIGNAL: track 0.00 -> 60.2 mm, vias 0 -> 2
- net BASE_LED: track 0.00 -> 58.1 mm, vias 0 -> 2
- net RX: track 0.00 -> 56.0 mm, vias 0 -> 2
- net A_AUX: track 0.00 -> 50.8 mm, vias 0 -> 2
- net D_AUX: track 0.00 -> 50.4 mm, vias 0 -> 2
- net TX: track 0.00 -> 48.3 mm, vias 0 -> 2
- net FOREARM_LED: track 0.00 -> 40.9 mm, vias 0 -> 2
- net SHOULDER_PWM1: track 0.00 -> 38.4 mm, vias 0 -> 2
- net +12V: track 28.5 -> 66.8 mm
- net GRIP_LED: track 0.00 -> 37.2 mm, vias 0 -> 2
- net GRIP_PWM: track 0.00 -> 36.9 mm, vias 0 -> 2
- net N$29: track 0.00 -> 36.9 mm, vias 0 -> 2
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
Commit message: everything done except ground planes
Parts:
- S2: value ENCODER_EVEJB -> ACZ11BR1E-20FA1; device devon:EVEJB -> devon:ACZ11BR1E-20FA1-20C
- S3: value S_BUTTON_TACTILE_PTS645 -> S_BUTTON_TACTILE_KT11S1SA2M35LFG; device devon:PTS645-SMD -> devon:C&K_SA2M_SA1M
- moved S1 13.9 mm to (6.50, 52.0), turned to 0 degrees
- moved C20 11.6 mm to (20.1, 48.3), turned to 270 degrees
- moved RN3 11.5 mm to (16.7, 48.3), turned to 90 degrees
- moved C21 11.2 mm to (13.1, 48.3), turned to 270 degrees
- moved R20 10.0 mm to (19.6, 45.3), turned to 180 degrees
- moved S3 8.24 mm to (21.5, 55.9)
- moved S2 2.15 mm to (8.50, 59.5), turned to 0 degrees
- moved J1 1.50 mm to (9.00, 46.4)
- moved RN2 1.00 mm to (13.8, 41.6)
Connections:
- removed net D11/MOSI: J1.4
- removed net D12/MISO: J1.1
- removed net D13/SCK: J1.3
- new net N$37: S1.2
- new net N$38: S1.4
- net +5V: now also RN3.1A, RN3.2A; no longer RN3.1B, RN3.4B, S3.1, S3.2
- net BUTTON: now also S3.2; no longer S3.3, S3.4
- net ENCODER_A: now also RN3.3A; no longer RN3.3B
- net ENCODER_B: now also RN3.4A; no longer RN3.2A
- net ENCODER_SW: now also S2.SW2; no longer S2.SW\
- net GND: now also S1.1, S2.GND, S2.SW1, S3.FRONT, S3.SIDE1, S3.SIDE2; no longer S1.3, S1.4, S2.GND_1, S2.GND_2
- net GRIP_LED: now also J1.1
- net GRIP_PWM: now also J1.4
- net N$34: now also RN3.4B; no longer RN3.4A
- net N$36: now also RN3.1B, RN3.3B; no longer RN3.1A, RN3.3A
- net RESET: now also S1.3; no longer S1.1, S1.2
- net STAT: now also J1.3
Routing:
- net +5V: track 189.1 -> 251.1 mm, vias 6 -> 10
- net STEP: track 1.97 -> 44.3 mm, vias 1 -> 4
- net GND: track 186.4 -> 225.0 mm, vias 19 -> 18
- net DIR: track 1.50 -> 39.7 mm, vias 1 -> 2
- net GRIP_LED: track 37.2 -> 71.5 mm
- net GRIP_PWM: track 36.9 -> 67.9 mm, vias 2 -> 3
- net STAT: track 13.0 -> 41.6 mm, vias 2 -> 3
- net ENCODER_SW: track 0.00 -> 28.5 mm
- net RESET: track 32.3 -> 54.3 mm, vias 2 -> 3
- net ENABLE: track 1.66 -> 22.8 mm, vias 1 -> 2
- net BUTTON: track 4.26 -> 24.2 mm
- net N$36: track 0.00 -> 19.8 mm
- net N$34: track 0.00 -> 18.6 mm
- net ENCODER_A: track 0.00 -> 16.8 mm, vias 0 -> 2
- net ENCODER_B: track 0.00 -> 12.1 mm
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
Commit message: All routing and positioning done
Parts:
- moved S3 0.51 mm to (22.0, 56.0)
- moved S2 0.50 mm to (9.00, 59.5)
- turned S1 to 180 degrees
Routing:
- net GND: track 225.0 -> 294.0 mm, vias 18 -> 33
- net RESET: track 54.3 -> 66.1 mm
- net +5V: track 251.1 -> 251.7 mm
- net N$34: track 18.6 -> 19.1 mm

Commit message: Entire board up for review
Routing:
- net GND: track 294.0 -> 295.4 mm
Other:
- board size 160 x 80 mm -> 50 x 65 mm
- board text added: "ICSP"
- board text added: "RESET"
- board text added: "STEPPER"

Commit message: Design Review 1, Solved all DRC errors
Parts:
- moved S2 2.00 mm to (9.00, 61.5)
- moved S1 1.00 mm to (6.50, 53.0)
- moved J2 0.50 mm to (45.0, 4.00)
- moved S3 0.50 mm to (22.0, 56.5)
Connections:
- net +5V: now also S3.1
Routing:
- net GND: track 295.4 -> 273.1 mm, vias 33 -> 34
- net +5V: track 251.7 -> 262.7 mm
- net RESET: track 66.1 -> 56.2 mm
- net STEP: track 44.3 -> 50.0 mm
- net ENCODER_SW: track 28.2 -> 29.7 mm
- net HALL_SIGNAL: track 60.0 -> 61.3 mm
- net N$36: track 19.6 -> 20.4 mm
- net BUTTON: track 24.3 -> 25.0 mm
- net N$34: track 19.1 -> 19.8 mm
- net N$54: track 16.5 -> 17.1 mm
- net N$11: track 6.43 -> 5.84 mm
Other:
- outline, holes or cut-outs redrawn
- board text added: "BY DEVON COPELAND"
- board text added: "ROBOT ARM CONTROLLER"

Commit message: gerber files
Parts:
- RN1: value 330K -> 330
- moved C2 0.20 mm to (10.1, 3.00)
Connections:
- net GND: now also P1.5; no longer P1.1
- net N$66: now also P1.4; no longer P1.2
- net N$8: now also P1.2; no longer P1.4
- net VUSB: now also P1.1; no longer P1.5
Routing:
- net N$8: track 7.35 -> 19.2 mm
- net RESET: track 56.2 -> 66.7 mm
- net VUSB: track 18.0 -> 10.9 mm
- net GND: track 273.1 -> 267.8 mm, vias 34 -> 35
- removed copper zone on layer 1, net N$52
Other:
- board text added: "DESIGNED BY DEVON COPELAND"
