File: Projects/Robot Arm/Robot Arm Controller.sch (EAGLE design)
At the start: 71 parts, among them IC1 U_FTDICHIP_FT232RL, J1 ICSP HEADER, J2 SERVO PWR, J3 STEPPER, J4 J_MOLEX_502386, P1 P_USB_MINIUX60A-MB-5ST, P2 +12V INPUT, Q1 FDV303N, U1 UA78M05CDCY, U2 TPS71550DCKR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

Commit message: Entire board up for review
Other:
- note added: "1.2"
- note removed: "1.1"
Changed lines of the file:
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@@
 <plain>
 <text x="223.52" y="-175.26" size="2.54" layer="94">A</text>
-<text x="241.3" y="-175.26" size="2.54" layer="94">1.1</text>
+<text x="241.3" y="-175.26" size="2.54" layer="94">1.2</text>
 <text x="170.18" y="-157.48" size="2.54" layer="94">ROBOT ARM</text>
 <text x="187.96" y="-175.26" size="2.54" layer="94">0002</text>
@@
 <text x="187.96" y="-175.26" size="2.54" layer="94">0002</text>
 <text x="223.52" y="-175.26" size="2.54" layer="94">A</text>
-<text x="241.3" y="-175.26" size="2.54" layer="94">1.1</text>
+<text x="241.3" y="-175.26" size="2.54" layer="94">1.2</text>
 <text x="5.08" y="-177.8" size="1.778" layer="95">MICROSTEPPING CONFIGURABLE
 WITH R7, R8 AND R9: SEE DATASHEET</text>

Commit message: Design Review 1, Solved all DRC errors
Connections:
- net +5V: now also S3.1
Other:
- moved on the sheet: RN3A
Changed lines of the file:
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@@
 <wire x1="101.6" y1="-157.48" x2="104.14" y2="-157.48" width="0.1524" layer="91"/>
 <pinref part="GND9" gate="1" pin="GND"/>
+<junction x="104.14" y="-157.48"/>
+<junction x="104.14" y="-160.02"/>
 </segment>
 <segment>
@@
 <wire x1="60.96" y1="-165.1" x2="60.96" y2="-167.64" width="0.1524" layer="91"/>
 <pinref part="GND6" gate="1" pin="GND"/>
+<junction x="60.96" y="-165.1"/>
 </segment>
 </net>
@@
 <wire x1="66.04" y1="-109.22" x2="66.04" y2="-111.76" width="0.1524" layer="91"/>
 <junction x="27.94" y="-109.22"/>
+<junction x="66.04" y="-111.76"/>
 </segment>
 <segment>
@@
 <instance part="R17" gate="A" x="137.16" y="-167.64" rot="R270"/>
 <instance part="C20" gate="G$1" x="162.56" y="-83.82" rot="MR270"/>
-<instance part="RN3" gate="A" x="195.58" y="-73.66" rot="R90"/>
+<instance part="RN3" gate="A" x="195.58" y="-73.66" rot="R270"/>
 <instance part="RN3" gate="B" x="180.34" y="-73.66" rot="R270"/>
 <instance part="RN3" gate="C" x="203.2" y="-81.28" rot="MR0"/>
@@
 <pinref part="GND34" gate="1" pin="GND"/>
 <pinref part="Q1" gate="A" pin="SOURCE"/>
+<junction x="165.1" y="-53.34"/>
 </segment>
 <segment>
@@
 <wire x1="180.34" y1="-66.04" x2="187.96" y2="-66.04" width="0.1524" layer="91"/>
 <wire x1="187.96" y1="-66.04" x2="195.58" y2="-66.04" width="0.1524" layer="91"/>
-<wire x1="195.58" y1="-66.04" x2="195.58" y2="-78.74" width="0.1524" layer="91"/>
+<wire x1="195.58" y1="-66.04" x2="195.58" y2="-68.58" width="0.1524" layer="91"/>
 <wire x1="187.96" y1="-66.04" x2="187.96" y2="-60.96" width="0.1524" layer="91"/>
 <pinref part="P+23" gate="1" pin="+5V"/>
@@
 </segment>
 <segment>
-<wire x1="187.96" y1="-121.92" x2="182.88" y2="-121.92" width="0.1524" layer="91"/>
 <wire x1="182.88" y1="-121.92" x2="182.88" y2="-116.84" width="0.1524" layer="91"/>
 <pinref part="P+22" gate="1" pin="+5V"/>
+<pinref part="S3" gate="A" pin="1"/>
+<wire x1="182.88" y1="-121.92" x2="185.42" y2="-121.92" width="0.1524" layer="91"/>
 </segment>
 <segment>
@@
 <wire x1="195.58" y1="-81.28" x2="198.12" y2="-81.28" width="0.1524" layer="91"/>
 <pinref part="RN3" gate="A" pin="2"/>
-<wire x1="195.58" y1="-81.28" x2="195.58" y2="-68.58" width="0.1524" layer="91"/>
+<wire x1="195.58" y1="-81.28" x2="195.58" y2="-78.74" width="0.1524" layer="91"/>
 <junction x="195.58" y="-81.28"/>
 <pinref part="S2" gate="A" pin="A"/>
@@
 <wire x1="81.28" y1="-83.82" x2="81.28" y2="-73.66" width="0.1524" layer="91"/>
 <wire x1="81.28" y1="-73.66" x2="73.66" y2="-73.66" width="0.1524" layer="91"/>
+<junction x="73.66" y="-73.66"/>
 </segment>
 </net>
@@
 <pinref part="R13" gate="A" pin="1"/>
 <wire x1="101.6" y1="-83.82" x2="99.06" y2="-83.82" width="0.1524" layer="91"/>
+<junction x="101.6" y="-60.96"/>
 </segment>
 </net>
@@
 <segment>
 <pinref part="J4" gate="A" pin="13"/>
-<wire x1="215.9" y1="-45.72" x2="187.96" y2="-45.72" width="0.1524" layer="91"/>
 <label x="190.5" y="-45.72" size="1.778" layer="95"/>
 <wire x1="215.9" y1="-45.72" x2="187.96" y2="-45.72" width="0.1524" layer="91"/>
@@
 <label x="142.24" y="-38.1" size="1.778" layer="95"/>
 <pinref part="Q1" gate="A" pin="GATE"/>
-</segment>
-</net>
+<junction x="152.4" y="-38.1"/>
+</segment>
+</net>

Commit message: gerber files
Parts:
- RN1: value 330K -> 330
Changed lines of the file:
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@@
 <part name="LED2" library="devon" deviceset="D_LED" device="SML0805"/>
 <part name="Y1" library="devon" deviceset="G_RESONATOR" device="MU" value="CSTCE16M0V13"/>
-<part name="RN1" library="devon" deviceset="R_RESISTOR_NETWORK_EXB-V8V103JV" device="" value="330K"/>
+<part name="RN1" library="devon" deviceset="R_RESISTOR_NETWORK_EXB-V8V103JV" device="" value="330"/>
 <part name="GND15" library="devon-supply" deviceset="GND" device=""/>
 <part name="GND10" library="devon-supply" deviceset="GND" device=""/>
@@
 </sheet>
 </sheets>
+<errors>
+</errors>
 </schematic>
 </drawing>
